File: pcb/salo.brd (EAGLE design)
At the start: 12 parts, among them IC2 LT1763CS8-3.3

Commit message: Add 2x N-channel enhancement MOSFET, SO-8.
Parts:
- added LED1: LAP4-TOP, led:P47F-TOP
- added R1: 10k, rcl:R0805
- added T1: DMN3024LSD, zetex:SO8
Connections:
- new net N$2: R1.2, T1.2
- new net N$3: LED1.C, T1.7, T1.8
- net GND: now also R1.1, T1.1, T1.3
- net VCC: now also LED1.A, T1.5, T1.6
Changed lines of the file:
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@@
 <element name="R3" library="rcl" package="R0805" value="10k" x="55.499" y="24.8285" rot="R270"/>
 <element name="R4" library="rcl" package="R0805" value="10k" x="55.499" y="21.2725" rot="R270"/>
+<element name="T1" library="zetex" package="SO8" value="DMN3024LSD" x="30.48" y="0">
+<attribute name="OC_FARNELL" value="unknown" x="30.48" y="0" size="1.778" layer="27" display="off"/>
+<attribute name="MPN" value="" x="30.48" y="0" size="1.778" layer="27" display="off"/>
+<attribute name="MF" value="" x="30.48" y="0" size="1.778" layer="27" display="off"/>
+<attribute name="OC_NEWARK" value="unknown" x="30.48" y="0" size="1.778" layer="27" display="off"/>
+</element>
+<element name="R1" library="rcl" package="R0805" value="10k" x="27.94" y="-7.62"/>
+<element name="LED1" library="led" package="P47F-TOP" value="LAP4-TOP" x="30.48" y="-15.24"/>
 </elements>
 <signals>
@@
 <wire x1="62.611" y1="19.4335" x2="62.291" y2="19.1135" width="0.254" layer="1"/>
 <via x="58.42" y="19.05" extent="1-16" drill="0.6"/>
+<contactref element="T1" pad="1"/>
+<contactref element="T1" pad="3"/>
+<contactref element="R1" pad="1"/>
+<wire x1="69.85" y1="16.51" x2="73.66" y2="24.13" width="0" layer="19" extent="1-1"/>
+<wire x1="62.611" y1="19.4335" x2="69.85" y2="16.51" width="0" layer="19" extent="1-1"/>
+<wire x1="58.42" y1="19.05" x2="62.291" y2="19.1135" width="0" layer="19" extent="1-1"/>
+<wire x1="55.499" y1="18.73" x2="58.42" y2="19.05" width="0" layer="19" extent="1-1"/>
+<wire x1="51.915" y1="18.47" x2="55.499" y2="18.73" width="0" layer="19" extent="1-1"/>
+<wire x1="62.611" y1="26.857" x2="62.611" y2="21.657" width="0" layer="19" extent="1-1"/>
+<wire x1="61.341" y1="26.857" x2="62.611" y2="26.857" width="0" layer="19" extent="1-1"/>
+<wire x1="31.115" y1="-2.6" x2="51.915" y2="18.47" width="0" layer="19" extent="1-1"/>
+<wire x1="28.575" y1="-2.6" x2="31.115" y2="-2.6" width="0" layer="19" extent="1-1"/>
+<wire x1="26.99" y1="-7.62" x2="28.575" y2="-2.6" width="0" layer="19" extent="1-1"/>
 </signal>
 <signal name="RTS">
@@
 <wire x1="63.948" y1="27.5082" x2="64.1258" y2="27.3304" width="0.4064" layer="1"/>
 <wire x1="64.1258" y1="27.3304" x2="65.0494" y2="27.3304" width="0.4064" layer="1"/>
+<contactref element="T1" pad="6"/>
+<contactref element="T1" pad="5"/>
+<contactref element="LED1" pad="A"/>
+<wire x1="32.385" y1="2.6" x2="65.024" y2="18.161" width="0" layer="19" extent="1-1"/>
+<wire x1="31.115" y1="2.6" x2="32.385" y2="2.6" width="0" layer="19" extent="1-1"/>
+<wire x1="28.03" y1="-15.24" x2="31.115" y2="2.6" width="0" layer="19" extent="1-1"/>
 </signal>
 <signal name="RESET">
@@
 <wire x1="50.27" y1="27.94" x2="49.53" y2="27.94" width="0.254" layer="16"/>
 </signal>
+<signal name="N$2">
+<contactref element="R1" pad="2"/>
+<contactref element="T1" pad="2"/>
+<wire x1="28.89" y1="-7.62" x2="29.845" y2="-2.6" width="0" layer="19" extent="1-1"/>
+</signal>
+<signal name="N$3">
+<contactref element="LED1" pad="C"/>
+<contactref element="T1" pad="7"/>
+<contactref element="T1" pad="8"/>
+<wire x1="28.575" y1="2.6" x2="29.845" y2="2.6" width="0" layer="19" extent="1-1"/>
+<wire x1="32.93" y1="-15.24" x2="29.845" y2="2.6" width="0" layer="19" extent="1-1"/>
+</signal>
 </signals>
